File: Hardware/Miguel's-Simple-Flight-Controller.kicad_sch (KiCad schematic)
At the start: 0 parts

Commit message: Schematic Done
Parts:
- added C1, C28, C29, C31: 1uF, symbol Device:C
- added C10, C11, C13, C17, C18: 22uF, symbol Device:C
- added C12, C2, C3, C5, C7, C8, C9: 10uF, symbol Device:C
- added C14, C15, C19, C20, C21, C22, C23, C24, C25, C26, C27, C37: 100nF, symbol Device:C
- added C16, C32: 2.2uF, symbol Device:C
- added C30: 1Uf, symbol Device:C
- added C33, C34: 20pF, symbol Device:C
- added C35, C36: 6.8pF, symbol Device:C
- added C4: 47nF, symbol Device:C
- added C6: 44uF, symbol Device:C
- added Card1: TF-01A, lcsc:TF-SMD_TF-01A, symbol lcsc:TF-01A
- added D1: LED, symbol Device:LED
- added J1: Screw_Terminal_01x02, symbol Connector:Screw_Terminal_01x02
- added J2, J3, J4, J5: Conn_01x03, symbol Connector_Generic:Conn_01x03
- added L1: L, symbol Device:L
- added L2: 1uH, symbol Device:L
- added L4: FCM1608KF-601T03, lcsc:L0603, symbol lcsc:FCM1608KF-601T03
- added L7: YHNR3015-5R6M, symbol Device:L
- added R1, R2: 5.1K, symbol Device:R
- added R10, R11, R12, R13, R16, R17, R18, R19, R20, R21, R22, R6, R7, R8, R9: 10K, symbol Device:R
- added R14: 100K, symbol Device:R
- added R15: 22.1K, symbol Device:R
- added R3: 383, symbol Device:R
- added R4: 5.23K, symbol Device:R
- added R5: 30.1K, symbol Device:R
- added SW1, SW2: TS-1088-AR02016, lcsc:SW-SMD_L3.9-W3.0-P4.45, symbol lcsc:TS-1088-AR02016
- added U1: BQ25883RGER, lcsc:VFQFPN-24_L4.0-W4.0-P0.50-BL-EP2.8, symbol lcsc:BQ25883RGER
- added U2: ICM-45686, lcsc:LGA-14_L3.0-W2.5-P0.50-TL, symbol lcsc:ICM-45686
- added U3: STM32F722RETx, Package_QFP:LQFP-64_10x10mm_P0.5mm, symbol MCU_ST_STM32F7:STM32F722RETx
- added U4: BMP580, lcsc:LGA-10_L2.0-W2.0-P0.50-TL_BMP580, symbol lcsc:BMP580
- added U5: TPS63070RNMR, lcsc:VQFN-HR-15_L3.0-W2.5-P0.50-BL_TPS63070RNMR, symbol lcsc:TPS63070RNMR
- added U6: LMR51430, Package_TO_SOT_SMD:SOT-23-6, symbol Regulator_Switching:LMR51430
- added USB1: TYPE-C 16PIN 2MD(073), lcsc:USB-C-SMD_TYPE-C-6PIN-2MD-073, symbol lcsc:TYPE-C16PIN2MD(073)
- added X1: X322525MOB4SI, lcsc:CRYSTAL-SMD_4P-L3.2-W2.5-BL, symbol lcsc:X322525MOB4SI
- added X2: Q13FC1350000400, lcsc:FC-135R_L3.2-W1.5, symbol lcsc:Q13FC1350000400
Connections:
- new net: C15.2, L7.1, U6.2 (SW)
- new net: R14.1, R15.1, U6.4 (FB)
- new net: C15.1, U6.6 (CB)
- new net: L4.1, U3.13 (VDDA)
- new net: C5.1, U1.21 (PMID), U1.22 (PMID)
- new net: R4.1, R5.2, R6.2, U1.7 (TS)
- new net: C32.1, U3.30 (VCAP_1)
- new net: D1.1 (K), U1.2 (STAT)
- new net: D1.2 (A), R7.1
- new net: L2.1, U5.11 (L1)
- new net: L2.2, U5.9 (L2)
- new net: C4.1, U1.12 (BTST)
- new net: R13.1, U5.2 (PG)
- new net: R13.2, U5.5 (FB)
- new net: C19.1, U4.1 (VDDIO)
- new net: C19.2, U4.5 (SDO)
- new net: R12.1, U5.1 (PS/SYNC), U5.14 (EN)
- new net: C14.2, U5.3 (Vaux)
- new net: R2.2, USB1.10 (CC2)
- new net: R1.2, USB1.4 (CC1)
- new net: L1.2, U1.17 (SW), U1.18 (SW)
- new net: R3.2, U1.8 (ILIM)
- new net +3.3V: C17.1, C18.1, C20.1, C21.1, C22.1, C23.1, C24.1, C25.1, C26.1, C27.1, C28.1, C29.1, C30.1, C31.1, Card1.4 (VDD), L4.2, L7.2, R10.1, R11.1, R14.2, R16.1, R17.1, R18.1, R19.1, R20.1, R21.1, R7.2, R8.2, R9.1, SW2.1, U2.5 (VDDIO), U2.8 (VDD), U3.1 (VBAT), U3.19 (VDD), U3.32 (VDD), U3.48 (VDD), U3.64 (VDD), U4.10 (VDD)
- new net +5V: C10.1, C11.1, C12.1, C13.1, J2.1 (Pin_1), J3.1 (Pin_1), J4.1 (Pin_1), J5.1 (Pin_1), U5.7 (Vout), U5.8 (Vout)
- new net BAT+: C2.1, J1.1 (Pin_1), U1.13 (BAT), U1.14 (BAT)
- new net BMP_INT: U4.7 (INT)
- new net BOOT: R22.1, SW2.2, U3.60 (BOOT0)
- new net BPM_INT: U3.62 (PB9)
- new net BQ_CE: U1.3 (~{CE}), U3.61 (PB8)
- new net BQ_INT: R11.2, U1.6 (~{INT}), U3.57 (PB5)
- new net BQ_PG: R8.1, U1.9 (~{PG})
- new net BQ_SCL: R10.2, U1.5 (SCL)
- new net BQ_SDA: R9.2, U1.4 (SDA)
- new net BTST: C4.2
- new net GND: C10.2, C11.2, C12.2, C13.2, C14.1, C16.2, C17.2, C18.2, C2.2, C20.2, C21.2, C22.2, C23.2, C24.2, C25.2, C26.2, C27.2, C28.2, C29.2, C3.1, C30.2, C31.2, C32.2, C33.2, C34.2, C35.2, C36.2, C37.1, C5.2, C6.2, C7.2, C8.2, C9.2, Card1.10 (GND), Card1.11 (GND), Card1.12 (GND), Card1.13 (GND), Card1.6 (VSS), J2.3 (Pin_3), J3.3 (Pin_3), J4.3 (Pin_3), J5.3 (Pin_3), L1.1, R1.1, R15.2, R2.1, R22.2, R3.1, R5.1, R6.1, SW1.1, U1.19 (GND), U1.20 (GND), U2.6 (GND), U3.12 (VSSA), U3.18 (VSS), U3.31 (VSS), U3.47 (VSS), U3.63 (VSS), U4.3 (VSS), U4.6 (CSB), U4.8 (VSS), U4.9 (VSS), U5.10 (PGND), U5.15 (Vsel), U5.4 (GND), U5.6 (FB2), U6.1 (GND), USB1.1 (GND), USB1.12 (GND), USB1.13 (SHELL), USB1.14 (SHELL), X1.2 (GND), X1.4 (GND)
- new net HSE_IN: C33.1, U3.5 (PH0), X1.1 (OSC1)
- new net HSE_OUT: C34.1, U3.6 (PH1), X1.3 (OSC2)
- new net I2C_SCL: U3.58 (PB6), U4.2 (SCK)
- new net I2C_SDA: U3.59 (PB7), U4.4 (SDI)
- new net ICM_CS: U2.12 (AP_CS), U3.20 (PA4)
- new net ICM_INT1: U2.4 (INT1/INT), U3.24 (PC4), U3.41 (PA8)
- new net ICM_INT2: U2.9 (INT2/FSYNC/CLKIN), U3.42 (PA9)
- new net ICM_SCK: U2.13 (AP_SCL/AP_SCLK), U3.21 (PA5)
- new net ICM_SDI: U2.14 (AP_SDA/AP_SDIO/AP_SDI), U3.23 (PA7)
- new net ICM_SDO: U2.1 (AP_SDO/AP_AD0), U3.22 (PA6)
- new net LSE_IN: C35.1, U3.3 (PC14), X2.1
- new net LSE_OUT: C36.1, U3.4 (PC15), X2.2
- new net MOTOR0: J2.2 (Pin_2), U3.14 (PA0)
- new net MOTOR1: J3.2 (Pin_2), U3.15 (PA1)
- new net MOTOR2: J4.2 (Pin_2), U3.16 (PA2)
- new net MOTOR3: J5.2 (Pin_2), U3.17 (PA3)
- new net PGND: C1.1, J1.2 (Pin_2)
- new net RESET: C37.2, SW1.2, U3.7 (NRST)
- new net SD_CD: Card1.9 (CD), U3.55 (PB3)
- new net SD_CLK: Card1.5 (CLK(SCLK)), R21.2, U3.53 (PC12)
- new net SD_CMD: Card1.3 (CMD(DI)), R20.2, U3.54 (PD2)
- new net SD_DAT0: Card1.7 (DAT0(D0)), R16.2, U3.39 (PC8)
- new net SD_DAT1: Card1.8 (DAT1(RSV)), R17.2, U3.40 (PC9)
- new net SD_DAT2: Card1.1 (DAT2(RSV)), R18.2, U3.51 (PC10)
- new net SD_DAT3: Card1.2 (CDDAT3(CS)), R19.2, U3.52 (PC11)
- new net USB_DN: U3.44 (PA11), USB1.5 (DN2), USB1.7 (DN1)
- new net USB_DP: U3.45 (PA12), USB1.6 (DP1), USB1.8 (DP2)
- new net VBUS: C1.2, U1.23 (VBUS), USB1.11 (VBUS), USB1.2 (VBUS)
- new net VREGN: C3.2, R4.2, U1.11 (REGN)
- new net VSYS: C16.1, C6.1, C7.1, C8.1, C9.1, U1.15 (SYS), U1.16 (SYS), U5.12 (Vin), U5.13 (Vin), U6.3 (VIN), U6.5 (EN)
- no-connect marks 0 -> 31
Other:
- title: (none) -> Miguel's Simple Flight Controller

Commit message: Schematic Pretty-Much Done
Just missing Footprint assignation
Parts:
- removed L1: L, symbol Device:L
- removed L2: 1uH, symbol Device:L
- removed L7: YHNR3015-5R6M, symbol Device:L
- added C38, C39, C40, C41, C42: 0.1uF, symbol Device:C
- added J10: Conn_01x20, Connector_PinHeader_2.54mm:PinHeader_1x20_P2.54mm_Vertical, symbol Connector_Generic:Conn_01x20
- added J6, J7, J8, J9: Conn_01x02, Connector_PinHeader_2.54mm:PinHeader_1x02_P2.54mm_Vertical, symbol Connector_Generic:Conn_01x02
- added L1: 1uH, lcsc:L2520, symbol lcsc:DFE252012F-1R0M=P2
- added L2: 1.5uH, lcsc:IND-SMD_L4.0-W4.0-A, symbol lcsc:XFL4020-152MEC
- added L3: 5.6uH, lcsc:IND-SMD_L3.0-W3.0, symbol lcsc:YHNR3015-5R6M
- added LED0, LED1, LED2, LED3: Conn_01x04, Connector_PinHeader_2.54mm:PinHeader_1x04_P2.54mm_Vertical, symbol Connector_Generic:Conn_01x04
- added PWR1: 16-213/GHC-YR1S1/3T, lcsc:LED0402-R-RD, symbol lcsc:16-213_GHC-YR1S1_3T
- added R23: 330, symbol Device:R
- added U7: 74AHCT1G125DCKRG4, lcsc:SC-70-5_L2.1-W1.3-P0.65-LS2.1-BR, symbol lcsc:74AHCT1G125DCKRG4
- D1: footprint (none) -> lcsc:LED0402-R-RD
- J1: footprint (none) -> TerminalBlock:TerminalBlock_Xinya_XY308-2.54-2P_1x02_P2.54mm_Horizontal
- J2, J3, J4, J5: footprint (none) -> Connector_PinHeader_2.54mm:PinHeader_1x03_P2.54mm_Vertical
- R1, R10, R11, R12, R13, R15, R16, R17, R18, R19, R2, R20, R21, R22, R4, R5, R6, R7, R8, R9: footprint (none) -> Resistor_SMD:R_0201_0603Metric
Connections:
- net +3.3V: now also J10.3 (Pin_3), L3.2, PWR1.1 (A)
- net +5V: now also C38.2, C39.2, C40.2, C41.2, C42.1, U7.5 (VCC)
- net GND: now also C42.2, J10.2 (Pin_2), L1.2, LED0.4 (Pin_4), LED1.4 (Pin_4), LED2.4 (Pin_4), LED3.4 (Pin_4), PWR1.2 (C), U7.1 (~{OE}), U7.3 (GND)
- net ICM_INT2: now also U3.25 (PB0)
- net PGND: now also J6.2 (Pin_2), J7.2 (Pin_2), J8.2 (Pin_2), J9.2 (Pin_2)
- net VBUS: now also J10.1 (Pin_1)
- net VSYS: now also J6.1 (Pin_1), J7.1 (Pin_1), J8.1 (Pin_1), J9.1 (Pin_1)
- net at C15.2, U6.2 (SW): now also L3.1
- net at U5.11 (L1): now also L2.1
- net at U5.9 (L2): now also L2.2
- net at U1.17 (SW), U1.18 (SW): now also L1.1
- net PC2: now reaches U3.10 (PC2)
- net PC2: now also J10.5 (Pin_5)
- net PC3: now reaches U3.11 (PC3)
- net PC3: now also J10.6 (Pin_6)
- net PC13: now reaches U3.2 (PC13)
- net PC13: now also J10.9 (Pin_9)
- net PB1: now reaches U3.26 (PB1)
- net PB1: now also J10.13 (Pin_13)
- net PB2: now reaches U3.27 (PB2)
- net PB2: now also J10.14 (Pin_14)
- net LVL_SHFT: now reaches U3.28 (PB10)
- net LVL_SHFT: now also U7.2 (A)
- net PB11: now reaches U3.29 (PB11)
- net PB11: now also J10.16 (Pin_16)
- net PB12: now reaches U3.33 (PB12)
- net PB12: now also J10.17 (Pin_17)
- net PB13: now reaches U3.34 (PB13)
- net PB13: now also J10.18 (Pin_18)
- net PB14: now reaches U3.35 (PB14)
- net PB14: now also J10.19 (Pin_19)
- net PB15: now reaches U3.36 (PB15)
- net PB15: now also J10.20 (Pin_20)
- net PC6: now reaches U3.37 (PC6)
- net PC6: now also J10.7 (Pin_7)
- net PC7: now reaches U3.38 (PC7)
- net PC7: now also J10.8 (Pin_8)
- net LED: now reaches U3.43 (PA10)
- net PB4: now reaches U3.56 (PB4)
- net PB4: now also J10.15 (Pin_15)
- net PC1: now reaches U3.9 (PC1)
- net PC1: now also J10.4 (Pin_4)
- new net: R23.2, U7.4 (Y)
- new net: C41.1, LED1.1 (Pin_1)
- new net: C38.1, LED2.1 (Pin_1)
- new net: C40.1, LED0.1 (Pin_1)
- new net: C39.1, LED3.1 (Pin_1)
- new net LED0: LED0.2 (Pin_2), R23.1
- new net LED1: LED0.3 (Pin_3), LED1.2 (Pin_2)
- new net LED2: LED1.3 (Pin_3), LED2.2 (Pin_2)
- new net LED3: LED2.3 (Pin_3), LED3.2 (Pin_2)
- new net PA13: J10.10 (Pin_10)
- new net PA14: J10.11 (Pin_11)
- new net PA15: J10.12 (Pin_12)
- no-connect marks 31 -> 13
Other:
- moved on the sheet: C23, C24, C25, C26, C27, C28, C29, C30, C31, J2, J3, J4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

Commit message: Started on PCB
Parts:
- removed J1: Screw_Terminal_01x02, TerminalBlock:TerminalBlock_Xinya_XY308-2.54-2P_1x02_P2.54mm_Horizontal, symbol Connector:Screw_Terminal_01x02
- removed J10: Conn_01x20, Connector_PinHeader_2.54mm:PinHeader_1x20_P2.54mm_Vertical, symbol Connector_Generic:Conn_01x20
- added J1, J10, J12, J13: Conn_01x05, Connector_PinHeader_2.54mm:PinHeader_1x05_P2.54mm_Vertical, symbol Connector_Generic:Conn_01x05
- added J11: Conn_01x04, Connector_PinHeader_2.54mm:PinHeader_1x04_P2.54mm_Vertical, symbol Connector_Generic:Conn_01x04
- added R24: 44, Resistor_SMD:R_0201_0603Metric, symbol Device:R
- added U8: XT60, lcsc:CONN-TH_XT60, symbol lcsc:XT60
- C1, C12, C14, C15, C16, C19, C2, C20, C21, C22, C23, C24, C25, C26, C27, C28, C29, C3, C30, C31, C32, C33, C34, C35, C36, C37, C38, C39, C4, C40, C41, C42, C5, C7, C8, C9: footprint (none) -> Capacitor_SMD:C_0402_1005Metric
- C10, C11, C13, C17, C18, C6: footprint (none) -> Capacitor_SMD:C_0805_2012Metric
- R14: footprint (none) -> Resistor_SMD:R_0402_1005Metric
- R23, R3: footprint (none) -> Resistor_SMD:R_0201_0603Metric
Connections:
- net BPM_INT is gone; now on net BMP_INT: U3.62 (PB9)
- net +3.3V: now also J1.3 (Pin_3), R24.1; no longer PWR1.1 (A)
- net +5V: now also J11.2 (Pin_2)
- net BAT+: now also U8.2 (+)
- net GND: now also J1.2 (Pin_2), J11.1 (Pin_1)
- net PA13: now also U3.46 (PA13), J10.5 (Pin_5)
- net PA14: now also U3.49 (PA14), J12.1 (Pin_1)
- net PA15: now also U3.50 (PA15), J12.2 (Pin_2)
- net PB1: now also J12.3 (Pin_3)
- net PB11: now also J13.1 (Pin_1)
- net PB12: now also J13.2 (Pin_2)
- net PB13: now also J13.3 (Pin_3)
- net PB14: now also J13.4 (Pin_4)
- net PB15: now also J13.5 (Pin_5)
- net PB2: now also J12.4 (Pin_4)
- net PB4: now also J12.5 (Pin_5)
- net PC1: now also J10.1 (Pin_1)
- net PC13: now also J10.4 (Pin_4)
- net PC2: now also J10.2 (Pin_2)
- net PC3: now also J10.3 (Pin_3)
- net PC6: now also J11.3 (Pin_3)
- net PC7: now also J11.4 (Pin_4)
- net PGND: now also U8.1 (-)
- net VBUS: now also J1.1 (Pin_1)
- net VSYS: now also R12.2
- net PC0: now reaches U3.8 (PC0)
- net PC0: now also J1.5 (Pin_5)
- net LED renamed PA10
- net PA10: now also J1.4 (Pin_4)
- new net: PWR1.1 (A), R24.2
- no-connect marks 13 -> 12
Other:
- moved on the sheet: Card1, PWR1
